Commit message: Add world frame and link it to pelvis

File: src/atlas_description/urdf/atlas_v5.urdf (robot description, URDF)
Before this commit: robot drc_skeleton, 37 links, 36 joints
Links:
- added link world
Joints:
- added joint fix_pelvis_to_world: type None, parent world, child pelvis, origin xyz=0 0 0 rpy=0 0 0

Commit message: fixed (double meaning heh)

File: src/atlas_description/urdf/atlas_v5.urdf (robot description, URDF)
Before this commit: robot drc_skeleton, 38 links, 37 joints
Joints:
- joint fix_pelvis_to_world: type None -> fixed

Commit message: Get rid of atlas_v5 change

File: src/atlas_description/urdf/atlas_v5.urdf (robot description, URDF)
Before this commit: robot drc_skeleton, 38 links, 37 joints
Links:
- removed link world
Joints:
- removed joint fix_pelvis_to_world
